File: board/board.kicad_sch (KiCad schematic)
At the start: 1 part

Commit message: imported legacy version
Parts:
- added J1: (no value), symbol board-rescue:013_PoE_rectified-put_on_edge
- added J2: (no value), symbol board-rescue:014_PoE_controlled-put_on_edge
- LOGO1: value Logo_Open_Hardware_Small -> (none); footprint Symbol:OSHW-Symbol_6.7x6mm_SilkScreen -> (none)
Connections:
- new net Controller/PG: J2.6 (PG)
- new net Controller/poe+_in: J1.3 (48V), J1.4 (48V)
- new net Controller/poe+_out: J2.3 (48V), J2.4 (48V)
- new net GND: J1.1 (GND), J1.2 (GND), J1.5 (GND), J2.1 (GND), J2.2 (GND), J2.5 (GND)
Other:
- removed sheet implementation
- added sheet Controller (Controller.kicad_sch)
- note removed: "Input connectors go here"
- note removed: "Output connectors go here"
