File: board/implementation.kicad_sch (KiCad schematic)
At the start: 0 parts

Commit message: added schematic and footprint from legacy project
Parts:
- added C1, C2: 47nF, Capacitor_SMD:C_0603_1608Metric, symbol Device:C_Small
- added C3: 1uF, Capacitor_SMD:C_1206_3216Metric, symbol Device:C_Small
- added Q1: PSMN5R2-60YL, Package_TO_SOT_SMD:LFPAK33, symbol Transistor_FET:PSMN5R2-60YL
- added R1: 49.9R, Resistor_SMD:R_0603_1608Metric, symbol Device:R_Small
- added R2: 118R, Resistor_SMD:R_0603_1608Metric, symbol Device:R_Small
- added R3, R4: 0R, Resistor_SMD:R_0603_1608Metric, symbol Device:R_Small
- added R5: 8.2R, Resistor_SMD:R_0603_1608Metric, symbol Device:R_Small
- added R6: 3.3k, Resistor_SMD:R_0603_1608Metric, symbol Device:R_Small
- added R7, R8: 100k, Resistor_SMD:R_0603_1608Metric, symbol Device:R_Small
- added U1: LT4275AIDDPBF-LT4275AIDDPBF, Package_DFN_QFN:DFN-10-1EP_3x3mm_P0.5mm_EP1.65x2.38mm, symbol parts:LT4275AIDDPBF-LT4275AIDDPBF-Auto-Intern
Connections:
- new net: R4.1, U1.2 (AUX)
- new net: Q1.4 (G), R6.1, U1.9 (HSGATE)
- new net: C2.1, R6.2
- new net: C1.1, R5.2, U1.10 (VPORT)
- new net: R2.1, U1.4 (RCLASS++/NC)
- new net: R3.1, U1.1 (*IEEEUVLO)
- new net: R8.2, U1.6 (*T2P/NC)
- new net: R1.1, U1.3 (RCLASS)
- new net GND: C1.2, C2.2, C3.2, R1.2, R2.2, R3.2, R4.2, U1.11 (EPAD), U1.5 (GND)
- new net PG: R7.2, U1.7 (PWRGD)
- new net poe+_in: Q1.5 (D), R5.1
- new net poe+_out: C3.1, Q1.1 (S), Q1.2 (S), Q1.3 (S), R7.1, R8.1, U1.8 (HSSRC)
