File: board/implementation.kicad_sch (KiCad schematic)
At the start: 13 parts, among them Q1 PSMN5R2-60YL, U1 LT4275AIDDPBF-LT4275AIDDPBF

Commit message: changed PSMN5R2 footprint from LFPAK33 to LFPAK56
The PSMN5R2 is not available in LFPAK33.
Parts:
- Q1: footprint Package_TO_SOT_SMD:LFPAK33 -> Package_TO_SOT_SMD:LFPAK56
Changed lines of the file:
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@@
     (property "Reference" "Q1" (id 0) (at 200.66 66.2432 90))
     (property "Value" "PSMN5R2-60YL" (id 1) (at 200.66 68.5546 90))
-    (property "Footprint" "Package_TO_SOT_SMD:LFPAK33" (id 2) (at 200.66 71.12 0)
+    (property "Footprint" "Package_TO_SOT_SMD:LFPAK56" (id 2) (at 200.66 71.12 0)
       (effects (font (size 1.27 1.27)) hide)
     )
